File: 1-WireThermocouple.brd (EAGLE design)
At the start: 40.1 x 18 mm, 15 parts, among them IC3 MCP1703, J2 RJ11-6PTH, Q1 BSS138, U1 MAX31850, X1 3.5mm, X2 RJ45-6L-B

Commit message: LDO footprint fixed
Parts:
- FB1, FB2: value Ferrite -> 470
- moved U$8 1.00 mm to (27.0, 9.00)
Connections:
- net 3.3V: now also C3.1, IC3.2; no longer C2.1, IC3.3
- net VIN: now also C2.1, IC3.3; no longer C3.1, IC3.2
Routing:
- net GND: track 41.6 -> 0.00 mm
- net VIN: track 11.6 -> 16.4 mm
- net 3.3V: track 30.9 -> 27.1 mm
- net OW: track 15.5 -> 14.8 mm
- added copper zone on layer 1, net GND
Other:
- board text added: "1-Wire Thermocouple v2"
- board text added: "Ferrite"
- board text added: "TaaraLabs.eu/tc2"
- board text removed: "1-Wire Thermocouple v1"
- board text removed: "TaaraLabs.eu/tc1"
