File: 1-WireThermocouple.sch (EAGLE design)
At the start: 13 parts, among them IC3 MCP1703, J2 RJ11-6PTH, Q1 BSS138, U1 MAX31850, X1 3.5mm, X2 RJ45-6L-B

Commit message: LDO footprint fixed
Parts:
- FB1, FB2: value Ferrite -> 470
Connections:
- net 3.3V: now also C3.1, IC3.VO; no longer C2.1, IC3.VI
- net VIN: now also C2.1, IC3.VI; no longer C3.1, IC3.VO
